File: UINIO-Storage.kicad_pcb (KiCad board)
At the start: 2 copper layers, 36.3 x 54 mm, 30 parts, among them J1 Conn_01x04_Pin, J2 Conn_01x04_Pin, J3 Conn_01x06_Pin, J4 Conn_01x06_Pin, U1 I2C-24-EEPROM-SOIC8, U2 I2C-24-EEPROM-TSSOP8, U3 SPI-25-Flash-SOIC8, U4 ME6211

Commit message: Finish schematic diagram.
Other:
- outline, holes or cut-outs redrawn
- board text added: "EEPROM SOIC8"
- board text added: "EEPROM TSSOP8"
- board text added: "Flash SOIC8"
- board text added: "SPI MicroSD"

Commit message: Commit PCB layout.
Parts:
- added C4: 0.1uF, Capacitor_SMD:C_0402_1005Metric, F.Cu at (157.4, 114.0)
- added D5: LED Red, LED_SMD:LED_0603_1608Metric, F.Cu at (147.7, 114.3)
- added J5: Conn_01x06_Pin, Connector_PinHeader_2.54mm:PinHeader_1x06_P2.54mm_Vertical, F.Cu at (145.5, 123.6)
- added R13: 2K, Resistor_SMD:R_0402_1005Metric, F.Cu at (145.4, 113.7)
- added U5: SPI-25-Flash-WSON8, Package_SON:WSON-8-1EP_6x5mm_P1.27mm_EP3.4x4.3mm, F.Cu at (152.8, 115.4)
- moved J3 68.9 mm to (178.2, 88.9), turned to 0 degrees
- moved C5 64.0 mm to (128.7, 88.6), turned to -90 degrees
- moved D1 63.3 mm to (170.1, 89.1), turned to 180 degrees
- moved U4 61.9 mm to (131.7, 88.7), turned to 180 degrees
- moved R5 61.7 mm to (167.1, 89.2), turned to 180 degrees
- moved C6 60.3 mm to (134.8, 88.6), turned to 90 degrees
- moved R11 58.3 mm to (131.0, 92.0), turned to 0 degrees
- moved R9 55.8 mm to (131.0, 94.0), turned to 0 degrees
- moved J4 54.5 mm to (123.0, 101.3), turned to 180 degrees
- moved U3 54.3 mm to (168.9, 95.5), turned to -90 degrees
- moved R10 53.3 mm to (131.0, 96.1), turned to 0 degrees
- moved R8 50.8 mm to (131.0, 98.1), turned to 0 degrees
- moved Card1 48.7 mm to (142.0, 94.9), turned to 90 degrees
- moved R12 48.4 mm to (131.0, 100.1), turned to 0 degrees
- moved C1 47.5 mm to (170.3, 101.8), turned to 180 degrees
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Other:
- board size 36.3 x 54 mm -> 58 x 39.5 mm
- board text added: "EEPROM SOIC"
- board text added: "EEPROM TSSOP"
- board text added: "Flash SOIC"
- board text added: "Flash WSON"
- board text removed: "EEPROM SOIC8"
- board text removed: "EEPROM TSSOP8"
- board text removed: "Flash SOIC8"
- board text removed: "UINIO-Storage"
- board text removed: "Version 1.0.0"
