File: UINIO-Storage.kicad_sch (KiCad schematic)
At the start: 35 parts, among them J1 Conn_01x04_Pin, J2 Conn_01x04_Pin, J3 Conn_01x06_Pin, J4 Conn_01x06_Pin, J5 Conn_01x06_Pin, U1 I2C-24-EEPROM-SOIC8, U2 I2C-24-EEPROM-TSSOP8, U3 SPI-25-Flash-SOIC8, U4 ME6211, U5 SPI-25-Flash-WSON8

Commit message: Finish PCB Layout.
Parts:
- removed J4: Conn_01x06_Pin, Connector_PinHeader_2.54mm:PinHeader_1x06_P2.54mm_Vertical, symbol Connector:Conn_01x06_Pin
- added J4: Conn_01x08_Pin, Connector_PinHeader_2.54mm:PinHeader_1x08_P2.54mm_Vertical, symbol Connector:Conn_01x08_Pin
- added R?: 10K, Resistor_SMD:R_0603_1608Metric, symbol Uinio:RES_0402
Connections:
- net EEPROM-SOIC8-SCL: now also J1.2 (Pin_2); no longer J1.3 (Pin_3)
- net EEPROM-SOIC8-SDA: now also J1.3 (Pin_3); no longer J1.2 (Pin_2)
- net EEPROM-TSSOP8-SCL: now also J2.2 (Pin_2); no longer J2.3 (Pin_3)
- net EEPROM-TSSOP8-SDA: now also J2.3 (Pin_3); no longer J2.2 (Pin_2)
- net Flash-SOIC8-CLK: now also J3.5 (Pin_5); no longer J3.4 (Pin_4)
- net Flash-SOIC8-CS: now also J3.2 (Pin_2); no longer J3.5 (Pin_5)
- net Flash-SOIC8-MISO: now also J3.3 (Pin_3); no longer J3.2 (Pin_2)
- net Flash-SOIC8-MOSI: now also J3.4 (Pin_4); no longer J3.3 (Pin_3)
- net Flash-WSON8-CLK: now also J5.3 (Pin_3); no longer J5.4 (Pin_4)
- net Flash-WSON8-CS: now also J5.4 (Pin_4); no longer J5.5 (Pin_5)
- net Flash-WSON8-MISO: now also J5.5 (Pin_5); no longer J5.2 (Pin_2)
- net Flash-WSON8-MOSI: now also J5.2 (Pin_2); no longer J5.3 (Pin_3)
- net SD-3.3V: now also R?.1; no longer C?.2, Card?.4 (VDD), R12.1, U4.5 (Vout)
- net SD-GND: no longer C?.1, C?.1, Card?.6 (VSS), D4.1 (K), U4.2 (Vss)
- net SDIO-2: now reaches Card?.1 (DAT2)
- net SDIO-2: now also R?.2, J4.2 (Pin_2)
- net SDIO1: now reaches Card?.8 (DAT1)
- net SDIO1: now also J4.7 (Pin_7), R?.2
- net SD-5V renamed SPI/SDIO-5V
- net SPI/SDIO-5V: now also J4.1 (Pin_1)
- net SD-CS renamed SPI-CS/SDIO-3
- net SPI-CS/SDIO-3: now also R?.2, J4.3 (Pin_3); no longer R?.2
- net SD-MISO renamed SPI-MISO/SDIO-0
- net SPI-MISO/SDIO-0: now also R?.2, J4.6 (Pin_6); no longer R?.2
- net SD-MOSI renamed SPI-MOSI/SDIO-CMD
- net SPI-MOSI/SDIO-CMD: now also R?.2, J4.4 (Pin_4); no longer R?.2
- net SD-SCLK renamed SPI/SDIO-SCLK
- net SPI/SDIO-SCLK: now also J4.5 (Pin_5); no longer R?.2
- new net SPI/SDIO-3.3V: C?.2, Card?.4 (VDD), R12.1, U4.5 (Vout)
- new net SPI/SDIO-GND: C?.1, C?.1, Card?.6 (VSS), D4.1 (K), J4.8 (Pin_8), U4.2 (Vss)
- no-connect marks 4 -> 2
Other:
- moved on the sheet: C?, Card?, D4, R12, R?, U4

Commit message: Finish PCB Layout.
Connections:
- net SD-GND: no longer Card?.10 (GND), Card?.11 (GND), Card?.12 (GND), Card?.13 (GND)
- new net: Card?.10 (GND), Card?.11 (GND), Card?.12 (GND), Card?.13 (GND)
Other:
- moved on the sheet: C?, Card?, D4, J4, R12, R?, U4

Commit message: Finish PCB Layout.
Connections:
- net SD-3.3V is gone; now on net SPI/SDIO-3.3V: R?.1, R?.1, R?.1, R?.1, R?.1
- net SPI/SDIO-GND: now also Card?.10 (GND), Card?.11 (GND), Card?.12 (GND), Card?.13 (GND)
Other:
- moved on the sheet: Card?
Changed lines of the file:
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@@
   (junction (at 210.82 165.1) (diameter 0) (color 0 0 0 0)
   )
-  (junction (at 382.27 127) (diameter 0) (color 0 0 0 0)
+  (junction (at 373.38 127) (diameter 0) (color 0 0 0 0)
   )
   (junction (at 245.11 100.33) (diameter 0) (color 0 0 0 0)
@@
   (junction (at 369.57 60.96) (diameter 0) (color 0 0 0 0)
   )
-  (junction (at 382.27 129.54) (diameter 0) (color 0 0 0 0)
+  (junction (at 373.38 129.54) (diameter 0) (color 0 0 0 0)
   )
   (junction (at 245.11 33.02) (diameter 0) (color 0 0 0 0)
@@
   (junction (at 228.6 231.14) (diameter 0) (color 0 0 0 0)
   )
-  (junction (at 382.27 111.76) (diameter 0) (color 0 0 0 0)
+  (junction (at 373.38 111.76) (diameter 0) (color 0 0 0 0)
   )
   (junction (at 374.65 60.96) (diameter 0) (color 0 0 0 0)
@@
   (junction (at 172.72 50.8) (diameter 0) (color 0 0 0 0)
   )
-  (no_connect (at 355.6 129.54))
+  (no_connect (at 346.71 129.54))
   (no_connect (at 369.57 66.04))
   (wire (pts (xy 186.69 33.02) (xy 245.11 33.02))
@@
     (stroke (width 0) (type default))
   )
-  (wire (pts (xy 382.27 127) (xy 381 127))
+  (wire (pts (xy 373.38 127) (xy 372.11 127))
     (stroke (width 0) (type default))
   )
@@
     (stroke (width 0) (type default))
   )
-  (wire (pts (xy 382.27 127) (xy 382.27 129.54))
+  (wire (pts (xy 373.38 127) (xy 373.38 129.54))
     (stroke (width 0) (type default))
   )
@@
     (stroke (width 0) (type default))
   )
-  (wire (pts (xy 382.27 129.54) (xy 387.35 129.54))
+  (wire (pts (xy 373.38 129.54) (xy 378.46 129.54))
     (stroke (width 0) (type default))
   )
@@
     (stroke (width 0) (type default))
   )
-  (wire (pts (xy 355.6 111.76) (xy 332.74 111.76))
+  (wire (pts (xy 346.71 111.76) (xy 323.85 111.76))
     (stroke (width 0.254) (type default))
   )
@@
     (stroke (width 0) (type default))
   )
-  (wire (pts (xy 382.27 129.54) (xy 381 129.54))
+  (wire (pts (xy 373.38 129.54) (xy 372.11 129.54))
     (stroke (width 0) (type default))
   )
@@
     (stroke (width 0) (type default))
   )
-  (wire (pts (xy 330.2 121.92) (xy 355.6 121.92))
+  (wire (pts (xy 321.31 121.92) (xy 346.71 121.92))
     (stroke (width 0.254) (type default))
   )
@@
     (stroke (width 0) (type default))
   )
-  (wire (pts (xy 330.2 116.84) (xy 355.6 116.84))
+  (wire (pts (xy 321.31 116.84) (xy 346.71 116.84))
     (stroke (width 0.254) (type default))
   )
@@
     (stroke (width 0) (type default))
   )
-  (wire (pts (xy 332.74 127) (xy 355.6 127))
+  (wire (pts (xy 323.85 127) (xy 346.71 127))
     (stroke (width 0) (type default))
   )
@@
     (stroke (width 0) (type default))
   )
-  (wire (pts (xy 382.27 109.22) (xy 382.27 111.76))
+  (wire (pts (xy 373.38 109.22) (xy 373.38 111.76))
     (stroke (width 0) (type default))
   )
@@
     (stroke (width 0) (type default))
   )
-  (wire (pts (xy 382.27 111.76) (xy 382.27 127))
+  (wire (pts (xy 373.38 111.76) (xy 373.38 127))
     (stroke (width 0) (type default))
   )
@@
     (stroke (width 0) (type default))
   )
-  (wire (pts (xy 355.6 114.3) (xy 332.74 114.3))
+  (wire (pts (xy 346.71 114.3) (xy 323.85 114.3))
     (stroke (width 0.254) (type default))
   )
@@
     (stroke (width 0) (type default))
   )
-  (wire (pts (xy 355.6 119.38) (xy 332.74 119.38))
+  (wire (pts (xy 346.71 119.38) (xy 323.85 119.38))
     (stroke (width 0.254) (type default))
   )
@@
     (stroke (width 0) (type default))
   )
-  (wire (pts (xy 382.27 109.22) (xy 381 109.22))
+  (wire (pts (xy 373.38 109.22) (xy 372.11 109.22))
     (stroke (width 0) (type default))
   )
@@
     (stroke (width 0) (type default))
   )
-  (wire (pts (xy 355.6 124.46) (xy 332.74 124.46))
+  (wire (pts (xy 346.71 124.46) (xy 323.85 124.46))
     (stroke (width 0.254) (type default))
   )
@@
     (stroke (width 0) (type default))
   )
-  (wire (pts (xy 382.27 111.76) (xy 381 111.76))
+  (wire (pts (xy 373.38 111.76) (xy 372.11 111.76))
     (stroke (width 0) (type default))
   )
@@
     (stroke (width 0) (type default))
   )
-  (wire (pts (xy 332.74 109.22) (xy 355.6 109.22))
+  (wire (pts (xy 323.85 109.22) (xy 346.71 109.22))
     (stroke (width 0) (type default))
   )
@@
     (effects (font (size 1.27 1.27)) (justify right bottom))
   )
-  (label "SPI-MOSI{slash}SDIO-CMD" (at 332.74 114.3 0) (fields_autoplaced)
+  (label "SPI-MOSI{slash}SDIO-CMD" (at 323.85 114.3 0) (fields_autoplaced)
     (effects (font (size 1.27 1.27)) (justify left bottom))
   )
@@
     (effects (font (size 1.27 1.27)) (justify right bottom))
   )
-  (label "SPI{slash}SDIO-3.3V" (at 330.2 116.84 180) (fields_autoplaced)
-    (effects (font (size 1.27 1.27)) (justify right bottom))
-  )
-  (label "SDIO1" (at 332.74 127 0) (fields_autoplaced)
-    (effects (font (size 1.27 1.27)) (justify left bottom))
-  )
-  (label "SDIO-2" (at 332.74 109.22 0) (fields_autoplaced)
+  (label "SPI{slash}SDIO-3.3V" (at 321.31 116.84 180) (fields_autoplaced)
+    (effects (font (size 1.27 1.27)) (justify right bottom))
+  )
+  (label "SDIO1" (at 323.85 127 0) (fields_autoplaced)
+    (effects (font (size 1.27 1.27)) (justify left bottom))
+  )
+  (label "SDIO-2" (at 323.85 109.22 0) (fields_autoplaced)
     (effects (font (size 1.27 1.27)) (justify left bottom))
   )
@@
     (effects (font (size 1.27 1.27)) (justify left bottom))
   )
-  (label "SPI{slash}SDIO-SCLK" (at 332.74 119.38 0) (fields_autoplaced)
-    (effects (font (size 1.27 1.27)) (justify left bottom))
-  )
-  (label "SPI-MISO{slash}SDIO-0" (at 332.74 124.46 0) (fields_autoplaced)
+  (label "SPI{slash}SDIO-SCLK" (at 323.85 119.38 0) (fields_autoplaced)
+    (effects (font (size 1.27 1.27)) (justify left bottom))
+  )
+  (label "SPI-MISO{slash}SDIO-0" (at 323.85 124.46 0) (fields_autoplaced)
     (effects (font (size 1.27 1.27)) (justify left bottom))
   )
@@
     (effects (font (size 1.27 1.27)) (justify right bottom))
   )
-  (label "SPI{slash}SDIO-GND" (at 330.2 121.92 180) (fields_autoplaced)
+  (label "SPI{slash}SDIO-GND" (at 321.31 121.92 180) (fields_autoplaced)
     (effects (font (size 1.27 1.27)) (justify right bottom))
   )
@@
     (effects (font (size 1.27 1.27)) (justify right bottom))
   )
-  (label "SD-3.3V" (at 365.76 157.48 0) (fields_autoplaced)
+  (label "SPI{slash}SDIO-3.3V" (at 365.76 157.48 0) (fields_autoplaced)
     (effects (font (size 1.27 1.27)) (justify left bottom))
   )
@@
     (effects (font (size 1.27 1.27)) (justify left bottom))
   )
-  (label "SPI-CS{slash}SDIO-3" (at 332.74 111.76 0) (fields_autoplaced)
+  (label "SPI-CS{slash}SDIO-3" (at 323.85 111.76 0) (fields_autoplaced)
     (effects (font (size 1.27 1.27)) (justify left bottom))
   )
@@
     (effects (font (size 1.27 1.27)) (justify right bottom))
   )
-  (label "SD-GND" (at 387.35 127 0) (fields_autoplaced)
+  (label "SPI{slash}SDIO-GND" (at 378.46 129.54 0) (fields_autoplaced)
     (effects (font (size 1.27 1.27)) (justify left bottom))
   )
@@
     )
   )
-  (symbol (lib_id "Uinio:TF_Card_02A") (at 368.3 119.38 0) (unit 1)
-    (in_bom yes) (on_board yes) (dnp no)
-    (property "Reference" "Card?" (at 368.808 103.886 0)
-      (effects (font (size 1.27 1.27)))
-    )
-    (property "Value" "TF_Card_02A" (at 368.554 135.128 0)
-      (effects (font (size 1.27 1.27)))
-    )
-    (property "Footprint" "Uinio:TF-SMD_TF-02" (at 368.3 109.22 0)
-      (effects (font (size 1.27 1.27)) hide)
-    )
-    (property "Datasheet" "" (at 368.3 114.3 0)
-      (effects (font (size 1.27 1.27)) hide)
-    )
-    (property "SuppliersPartNumber" "C2889261" (at 368.3 119.38 0)
-      (effects (font (size 1.27 1.27)) hide)
-    )
-    (property "uuid" "std:d296a76a79c743a0bd4ab3714a928763" (at 368.3 119.38 0)
-      (effects (font (size 1.27 1.27)) hide)
-    )
+  (symbol (lib_id "Uinio:TF_Card_02A") (at 359.41 119.38 0) (unit 1)
+    (in_bom yes) (on_board yes) (dnp no)
+    (property "Reference" "Card?" (at 359.918 103.886 0)
+      (effects (font (size 1.27 1.27)))
+    )
+    (property "Value" "TF_Card_02A" (at 359.664 135.128 0)
+      (effects (font (size 1.27 1.27)))
+    )
+    (property "Footprint" "Uinio:TF-SMD_TF-02" (at 359.41 109.22 0)
+      (effects (font (size 1.27 1.27)) hide)
+    )
+    (property "Datasheet" "" (at 359.41 114.3 0)
+      (effects (font (size 1.27 1.27)) hide)
+    )
+    (property "SuppliersPartNumber" "C2889261" (at 359.41 119.38 0)
+      (effects (font (size 1.27 1.27)) hide)
+    )
+    (property "uuid" "std:d296a76a79c743a0bd4ab3714a928763" (at 359.41 119.38 0)
+      (effects (font (size 1.27 1.27)) hide)
+    )

Commit message: Release UINIO-Storage version 1.0.0.
Other:
- company: 电子技术博客 UinIO.com -> UinIO.com 电子实验室
- moved on the sheet: C?, Card?, D4, R12, U4
