File: UINIO-Storage.kicad_sch (KiCad schematic)
At the start: 36 parts, among them J1 Conn_01x04_Pin, J2 Conn_01x04_Pin, J3 Conn_01x06_Pin, J4 Conn_01x08_Pin, J5 Conn_01x06_Pin, U1 I2C-24-EEPROM-SOIC8, U2 I2C-24-EEPROM-TSSOP8, U3 SPI-25-Flash-SOIC8, U4 ME6211, U5 SPI-25-Flash-WSON8

Commit message: Release UINIO-Storage version 1.0.0.
Other:
- company: UinIO.com 电子实验室 -> UinIO.com 电子技术实验室
Changed lines of the file:
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@@
     (date "2024-01-07")
     (rev "Version 1.0.0")
-    (company "UinIO.com 电子实验室")
+    (company "UinIO.com 电子技术实验室")
   )
   (junction (at 172.72 120.65) (diameter 0) (color 0 0 0 0)
